Commit message: Working commit

File: fairino_description/urdf/fairino5_v6.urdf (robot description, URDF)
Before this commit: robot fairino5_v6_robot, 7 links, 6 joints
Links:
- added link base_footprint
Joints:
- added joint base_joint: type fixed, parent base_footprint, child base_link, origin xyz=0 0 0 rpy=0 0 0.785398

Commit message: bug fixes

File: fairino_description/urdf/fairino5_v6.urdf (robot description, URDF)
Before this commit: robot fairino5_v6_robot, 8 links, 7 joints
Links:
- added link fr5_angled_attach, mass 0.0
- added link fr5_attach, mass 0.0
- added link fr5_base; collision mesh filename=package://pr_description/meshes/collision/pbf_mirror.stl; visual mesh filename=package://pr_description/meshes/pbf_mirror.stl
- added link fr5_deg10_base; collision mesh filename=package://pr_description/meshes/collision/pbf_deg10.stl; visual mesh filename=package://pr_description/meshes/pbf_deg10.stl
- added link fr5_deg10_camera_attach, mass 0.0
- added link fr5_deg10_camera_base_link, mass 0.0
- added link fr5_deg10_camera_body_link, mass 0.072
- added link fr5_deg10_camera_link, mass 0.0
- added link fr5_deg20_base; collision mesh filename=package://pr_description/meshes/collision/pbf_deg20.stl; visual mesh filename=package://pr_description/meshes/pbf_deg20.stl
- added link fr5_deg20_camera_attach, mass 0.0
- added link fr5_deg20_camera_base_link, mass 0.0
- added link fr5_deg20_camera_body_link, mass 0.072
- added link fr5_deg20_camera_link, mass 0.0
- added link fr5_ee_tip_bolting, mass 0.0
- added link fr5_ft_ee_tip, mass 0.0
- added link fr5_opp_attach, mass 0.0
Joints:
- added joint fr5_angled_attach_jt: type fixed, parent fr5_base, child fr5_angled_attach, origin xyz=-0.053435 -0.053435 -0.0455 rpy=0 0 -2.356194490192345
- added joint fr5_attach_jt: type fixed, parent wrist3_link, child fr5_attach, origin xyz=0 0 0.1 rpy=0 0 1.5708
- added joint fr5_bolting_tip_jt: type fixed, parent fr5_base, child fr5_ee_tip_bolting, origin xyz=-0.1015 -2.5e-05 -0.2855 rpy=0 3.141592653589793 3.141592653589793
- added joint fr5_deg10_attach_jt: type fixed, parent fr5_angled_attach, child fr5_deg10_base
- added joint fr5_deg10_camera_jt: type fixed, parent fr5_deg10_base, child fr5_deg10_camera_attach, origin xyz=0.069261 0.0 -0.021919 rpy=-2.9670597283903604 0 1.5707963267948966
- added joint fr5_deg10_ee_camera_attach_jt: type fixed, parent fr5_deg10_camera_attach, child fr5_deg10_camera_body_link
- added joint fr5_deg10_ee_camera_base_jt: type fixed, parent fr5_deg10_camera_base_link, child fr5_deg10_camera_link, origin xyz=0.01085 0.009 0.021 rpy=0 0 0
- added joint fr5_deg10_ee_camera_jt: type fixed, parent fr5_deg10_camera_body_link, child fr5_deg10_camera_base_link, origin xyz=0 0.021 0.00835 rpy=1.5707963267948966 -1.5707963267948966 0.0
- added joint fr5_deg20_attach_jt: type fixed, parent fr5_opp_attach, child fr5_deg20_base
- added joint fr5_deg20_camera_jt: type fixed, parent fr5_deg20_base, child fr5_deg20_camera_attach, origin xyz=0.07011 -0.000747 -0.018489 rpy=-2.792526803190927 0 1.5707963267948966
- added joint fr5_deg20_ee_camera_attach_jt: type fixed, parent fr5_deg20_camera_attach, child fr5_deg20_camera_body_link
- added joint fr5_deg20_ee_camera_base_jt: type fixed, parent fr5_deg20_camera_base_link, child fr5_deg20_camera_link, origin xyz=0.01085 0.009 0.021 rpy=0 0 0
- added joint fr5_deg20_ee_camera_jt: type fixed, parent fr5_deg20_camera_body_link, child fr5_deg20_camera_base_link, origin xyz=0 0.021 0.00835 rpy=1.5707963267948966 -1.5707963267948966 0.0
- added joint fr5_ee_attach_jt: type fixed, parent fr5_attach, child fr5_base, origin rpy=3.141592653589793 0 0
- added joint fr5_ft_ee_tip_jt: type fixed, parent fr5_base, child fr5_ft_ee_tip, origin xyz=0 0 -0.0395 rpy=0 3.141592653589793 3.141592653589793
- added joint fr5_opp_attach_jt: type fixed, parent fr5_base, child fr5_opp_attach, origin xyz=0 0.072 -0.0455 rpy=0 0 1.5707963267948966
